File: out/kicad/ProjectShellac.kicad_pcb (KiCad board)
At the start: 2 copper layers, 250 parts, among them U101 L_PLUS PRECISION GAIN, U102 L_MINUS PRECISION GAIN, U103 L DIFF 4.00x, U201 R_PLUS PRECISION GAIN, U202 R_MINUS PRECISION GAIN, U203 R DIFF 4.00x, U3001 L ACTIVE LF EQ, U3002 L RECOVERY, U3501 R ACTIVE LF EQ, U3502 R RECOVERY, U401 L ISOLATION BUFFER, U402 R ISOLATION BUFFER, U501 L MODE BUFFER, U502 R MODE BUFFER, U700 L HP SECTION A, U720 L HP SECTION B, U750 R HP SECTION A, U770 R HP SECTION B, U8001 L THAT1646, U9001 R THAT1646

Commit message: wip(pcb): snapshot SR-043 native placement and mechanical audit
Parts:
- added MH1: MountingHole_3.2mm_M3, MountingHole:MountingHole_3.2mm_M3, F.Cu at (25.0, 28.0)
- added MH2: MountingHole_3.2mm_M3, MountingHole:MountingHole_3.2mm_M3, F.Cu at (235.0, 28.0)
- added MH3: MountingHole_3.2mm_M3, MountingHole:MountingHole_3.2mm_M3, F.Cu at (235.0, 152.0)
- added MH4: MountingHole_3.2mm_M3, MountingHole:MountingHole_3.2mm_M3, F.Cu at (25.0, 152.0)
- moved R214 214.6 mm to (223.4, 31.4)
- moved C35023 213.7 mm to (221.0, 59.2)
- moved TP3505 212.5 mm to (221.0, 80.3)
- moved R225 209.3 mm to (223.4, 37.1)
- moved C35022 207.6 mm to (213.8, 59.2)
- moved TP3504 206.3 mm to (213.8, 80.3)
- moved R213 206.1 mm to (215.2, 31.4)
- moved D90032 201.6 mm to (220.5, 137.7)
- moved R224 200.8 mm to (215.2, 37.1)
- moved TP3503 200.2 mm to (206.6, 80.3)
- moved R212 197.6 mm to (207.0, 31.4)
- moved D90031 197.4 mm to (212.3, 137.7)
- moved C35020 194.7 mm to (199.4, 59.2)
- moved C35025 193.8 mm to (199.4, 66.2)
- moved D90030 193.4 mm to (204.1, 137.7)
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Other:
- board outline added: 220 x 140 mm
- copper layers 2 -> 4

Commit message: AE-071A: migrate SCH101 product architecture and reconcile native PCB
Parts:
- removed R115, R116, R125, R126, R215, R216, R225, R226: 0R, Resistor_SMD:R_0805_2012Metric
- removed R501, R502: 4700, Resistor_SMD:R_0805_2012Metric
- removed U102: L_MINUS PRECISION GAIN, Package_SO:SOIC-8_3.9x4.9mm_P1.27mm
- removed U202: R_MINUS PRECISION GAIN, Package_SO:SOIC-8_3.9x4.9mm_P1.27mm
- removed U3002: L RECOVERY, Package_SO:SOIC-8_3.9x4.9mm_P1.27mm
- removed U3502: R RECOVERY, Package_SO:SOIC-8_3.9x4.9mm_P1.27mm
- removed U402: R ISOLATION BUFFER, Package_SO:SOIC-8_3.9x4.9mm_P1.27mm
- removed U502: R MODE BUFFER, Package_SO:SOIC-8_3.9x4.9mm_P1.27mm
- removed U720: L HP SECTION B, Package_SO:SOIC-8_3.9x4.9mm_P1.27mm
- removed U770: R HP SECTION B, Package_SO:SOIC-8_3.9x4.9mm_P1.27mm
- added C104: 100p, Capacitor_SMD:C_0805_2012Metric, F.Cu at (8.87, 13.2)
- added C191: 100n, Capacitor_SMD:C_0805_2012Metric, F.Cu at (8.87, 16.2)
- added C192: 100n, Capacitor_SMD:C_0805_2012Metric, F.Cu at (8.87, 19.2)
- added C193: 100n, Capacitor_SMD:C_0805_2012Metric, F.Cu at (8.87, 22.2)
- added C194: 100n, Capacitor_SMD:C_0805_2012Metric, F.Cu at (8.87, 25.3)
- added C204: 100p, Capacitor_SMD:C_0805_2012Metric, F.Cu at (13.3, 13.2)
- added C291: 100n, Capacitor_SMD:C_0805_2012Metric, F.Cu at (13.3, 16.2)
- added C292: 100n, Capacitor_SMD:C_0805_2012Metric, F.Cu at (13.3, 19.2)
- added C293: 100n, Capacitor_SMD:C_0805_2012Metric, F.Cu at (13.3, 22.2)
- added C294: 100n, Capacitor_SMD:C_0805_2012Metric, F.Cu at (13.3, 25.3)
- added H110: GAIN LOW 4-GANG, Connector_PinHeader_2.54mm:PinHeader_2x04_P2.54mm_Vertical, F.Cu at (8.94, 1.79)
- added H111: GAIN HIGH 4-GANG, Connector_PinHeader_2.54mm:PinHeader_2x04_P2.54mm_Vertical, F.Cu at (16.1, 1.79)
- added H112: GAIN DEFAULT / PARK, Connector_PinHeader_2.54mm:PinHeader_2x04_P2.54mm_Vertical, F.Cu at (23.2, 1.79)
- added H120: LOAD +47p L/R, Connector_PinHeader_2.54mm:PinHeader_2x02_P2.54mm_Vertical, F.Cu at (1.79, 1.79)
- added H121: LOAD BASE / PARK, Connector_PinHeader_2.54mm:PinHeader_2x02_P2.54mm_Vertical, F.Cu at (1.79, 8.94)
- added H122: LOAD +100p L/R, Connector_PinHeader_2.54mm:PinHeader_2x02_P2.54mm_Vertical, F.Cu at (1.79, 16.1)
- added R104: 23700, Resistor_SMD:R_0805_2012Metric, F.Cu at (17.7, 13.2)
- added R105: 23700, Resistor_SMD:R_0805_2012Metric, F.Cu at (17.7, 16.1)
- added R204: 23700, Resistor_SMD:R_0805_2012Metric, F.Cu at (17.7, 19.1)
- added R205: 23700, Resistor_SMD:R_0805_2012Metric, F.Cu at (17.7, 22.0)
- added R4002: 4700, Resistor_SMD:R_0805_2012Metric, F.Cu at (32.3, 0.97)
- added R4502: 4700, Resistor_SMD:R_0805_2012Metric, F.Cu at (32.3, 3.92)
- added TP506: MONO_R_LEG, TestPoint:TestPoint_Pad_D1.5mm, F.Cu at (31.8, 9.18)
- C101, C102, C201, C202: value 1n -> 47p
- C103, C203: value 220p -> 47p
- C7001, C7002, C7201, C7202, C7501, C7502, C7701, C7702: footprint Capacitor_SMD:C_0805_2012Metric -> Capacitor_THT:C_Rect_L7.2mm_W3.5mm_P5.00mm_FKS2_FKP2_MKS2_MKP2
- D80030, D80031, D80032, D80033, D90030, D90031, D90032, D90033: value 1N4004 -> S1G
- R112, R122, R212, R222: value 249 -> 999
- R113, R123, R213, R223: value 750 -> 332
- R114, R124, R214, R224: value 1910 -> 866
- U101: value L_PLUS PRECISION GAIN -> OPA1656
- U103: value L DIFF 4.00x -> OPA1655
- U201: value R_PLUS PRECISION GAIN -> OPA1656
- U203: value R DIFF 4.00x -> OPA1655
- U3001: value L ACTIVE LF EQ -> OPA1612
- U3501: value R ACTIVE LF EQ -> OPA1612
- U401: value L ISOLATION BUFFER -> OPA1656
- U501: value L MODE BUFFER -> OPA1656
- U700: value L HP SECTION A -> OPA1656
- U750: value R HP SECTION A -> OPA1656
Connections:
- net /SCH105 Channel Mode Matrix/MONO_AVG renamed ROOT__MONO_AVG
- C101 pad 1: Net-(U101-IN+) -> /SCH101 Balanced Input and Differential Conversion/SCH101_L_LOAD_POS
- C102 pad 2: Net-(U102-IN+) -> /SCH101 Balanced Input and Differential Conversion/SCH101_L_LOAD_NEG
- C103 pad 1: Net-(U102-IN+) -> /SCH101 Balanced Input and Differential Conversion/SCH101_L_LOAD_POS
- C103 pad 2: Net-(U101-IN+) -> /SCH101 Balanced Input and Differential Conversion/SCH101_L_LOAD47_BRANCH
- C201 pad 1: Net-(U201-IN+) -> /SCH101 Balanced Input and Differential Conversion/SCH101_R_LOAD_POS
- C202 pad 2: Net-(U202-IN+) -> /SCH101 Balanced Input and Differential Conversion/SCH101_R_LOAD_NEG
- C203 pad 1: Net-(U202-IN+) -> /SCH101 Balanced Input and Differential Conversion/SCH101_R_LOAD_POS
- C203 pad 2: Net-(U201-IN+) -> /SCH101 Balanced Input and Differential Conversion/SCH101_R_LOAD47_BRANCH
- C30051 pad 1: -18V -> 0VA
- C30051 pad 2: 0VA -> -18V
- C30053 pad 1: -18V -> 0VA
- C30053 pad 2: 0VA -> -18V
- C35051 pad 1: -18V -> 0VA
- C35051 pad 2: 0VA -> -18V
- C35053 pad 1: -18V -> 0VA
- C35053 pad 2: 0VA -> -18V
- C5092 pad 1: -18V -> 0VA
- C5092 pad 2: 0VA -> -18V
- C5094 pad 1: -18V -> 0VA
- C5094 pad 2: 0VA -> -18V
- C7002 pad 1: Net-(U700-IN) -> Net-(U700A-IN)
- C7202 pad 1: Net-(U720-IN) -> Net-(U700B-IN)
- C7502 pad 1: Net-(U750-IN) -> Net-(U750A-IN)
- C7702 pad 1: Net-(U770-IN) -> Net-(U750B-IN)
- C80041 pad 1: -18V -> 0VA
- C80041 pad 2: 0VA -> -18V
- C80043 pad 1: -18V -> 0VA
- C80043 pad 2: 0VA -> -18V
- C90041 pad 1: -18V -> 0VA
- C90041 pad 2: 0VA -> -18V
- C90043 pad 1: -18V -> 0VA
- C90043 pad 2: 0VA -> -18V
- R102 pad 2: Net-(U101-IN+) -> /SCH101 Balanced Input and Differential Conversion/SCH101_L_LOAD_POS
- R103 pad 2: Net-(U102-IN+) -> /SCH101 Balanced Input and Differential Conversion/SCH101_L_LOAD_NEG
- R111 pad 2: Net-(U101-FB-) -> /SCH101 Balanced Input and Differential Conversion/SCH101_L_PLUS_FB
- R112 pad 1: Net-(R112-Pad1) -> /SCH101 Balanced Input and Differential Conversion/SCH101_L_PLUS_FB
- R113 pad 1: Net-(R113-Pad1) -> /SCH101 Balanced Input and Differential Conversion/SCH101_L_LT5400_PLUS_SRC
- R113 pad 2: Net-(R112-Pad1) -> /SCH101 Balanced Input and Differential Conversion/SCH101_L_PLUS_LOW_BRANCH
- R114 pad 1: Net-(R114-Pad1) -> /SCH101 Balanced Input and Differential Conversion/SCH101_L_PLUS_FB
- R114 pad 2: Net-(R113-Pad1) -> /SCH101 Balanced Input and Differential Conversion/SCH101_L_PLUS_HIGH_BRANCH
- R121 pad 2: Net-(U102-FB-) -> /SCH101 Balanced Input and Differential Conversion/SCH101_L_MINUS_FB
- R122 pad 1: Net-(R122-Pad1) -> /SCH101 Balanced Input and Differential Conversion/SCH101_L_MINUS_FB
- R123 pad 1: Net-(R123-Pad1) -> /SCH101 Balanced Input and Differential Conversion/SCH101_L_LT5400_MINUS_SRC
- R123 pad 2: Net-(R122-Pad1) -> /SCH101 Balanced Input and Differential Conversion/SCH101_L_MINUS_LOW_BRANCH
- R124 pad 1: Net-(R124-Pad1) -> /SCH101 Balanced Input and Differential Conversion/SCH101_L_MINUS_FB
- R124 pad 2: Net-(R123-Pad1) -> /SCH101 Balanced Input and Differential Conversion/SCH101_L_MINUS_HIGH_BRANCH
- R202 pad 2: Net-(U201-IN+) -> /SCH101 Balanced Input and Differential Conversion/SCH101_R_LOAD_POS
- R203 pad 2: Net-(U202-IN+) -> /SCH101 Balanced Input and Differential Conversion/SCH101_R_LOAD_NEG
- R211 pad 2: Net-(U201-FB-) -> /SCH101 Balanced Input and Differential Conversion/SCH101_R_PLUS_FB
- R212 pad 1: Net-(R212-Pad1) -> /SCH101 Balanced Input and Differential Conversion/SCH101_R_PLUS_FB
- R213 pad 1: Net-(R213-Pad1) -> /SCH101 Balanced Input and Differential Conversion/SCH101_R_LT5400_PLUS_SRC
- R213 pad 2: Net-(R212-Pad1) -> /SCH101 Balanced Input and Differential Conversion/SCH101_R_PLUS_LOW_BRANCH
- R214 pad 1: Net-(R214-Pad1) -> /SCH101 Balanced Input and Differential Conversion/SCH101_R_PLUS_FB
- R214 pad 2: Net-(R213-Pad1) -> /SCH101 Balanced Input and Differential Conversion/SCH101_R_PLUS_HIGH_BRANCH
- R221 pad 2: Net-(U202-FB-) -> /SCH101 Balanced Input and Differential Conversion/SCH101_R_MINUS_FB
- R222 pad 1: Net-(R222-Pad1) -> /SCH101 Balanced Input and Differential Conversion/SCH101_R_MINUS_FB
- R223 pad 1: Net-(R223-Pad1) -> /SCH101 Balanced Input and Differential Conversion/SCH101_R_LT5400_MINUS_SRC
- R223 pad 2: Net-(R222-Pad1) -> /SCH101 Balanced Input and Differential Conversion/SCH101_R_MINUS_LOW_BRANCH
- R224 pad 1: Net-(R224-Pad1) -> /SCH101 Balanced Input and Differential Conversion/SCH101_R_MINUS_FB
- R224 pad 2: Net-(R223-Pad1) -> /SCH101 Balanced Input and Differential Conversion/SCH101_R_MINUS_HIGH_BRANCH
- R30040 pad 1: Net-(U3002-FB-) -> Net-(U3001B-FB-)
- R30041 pad 2: Net-(U3002-FB-) -> Net-(U3001B-FB-)
- R35040 pad 1: Net-(U3502-FB-) -> Net-(U3501B-FB-)
- R35041 pad 2: Net-(U3502-FB-) -> Net-(U3501B-FB-)
- R4001 pad 1: Net-(U401-OUT) -> Net-(U401A-IN-)
- R4501 pad 1: Net-(U402-OUT) -> Net-(U401B-IN-)
- R510 pad 1: Net-(U501-IN) -> Net-(U501A-IN)
- R511 pad 1: Net-(U501-OUT) -> Net-(U501A-IN-)
- R520 pad 1: Net-(U502-IN) -> Net-(U501B-IN)
- R521 pad 1: Net-(U502-OUT) -> Net-(U501B-IN-)
- R7002 pad 2: Net-(U700-IN) -> Net-(U700A-IN)
- R7202 pad 2: Net-(U720-IN) -> Net-(U700B-IN)
- R7502 pad 2: Net-(U750-IN) -> Net-(U750A-IN)
- R7702 pad 2: Net-(U770-IN) -> Net-(U750B-IN)
- U101 pad 1: Net-(U101-IN+) -> /SCH101 Balanced Input and Differential Conversion/SCH101_L_LT5400_PLUS_SRC
- U101 pad 2: Net-(U101-FB-) -> /SCH101 Balanced Input and Differential Conversion/SCH101_L_PLUS_FB
- U101 pad 3: /SCH101 Balanced Input and Differential Conversion/SCH101_L_LT5400_PLUS_SRC -> /SCH101 Balanced Input and Differential Conversion/SCH101_L_LOAD_POS
- U101 pad 4: +18V -> -18V
- U101 pad 5: -18V -> /SCH101 Balanced Input and Differential Conversion/SCH101_L_LOAD_NEG
- U101 pad 6: (no net) -> /SCH101 Balanced Input and Differential Conversion/SCH101_L_MINUS_FB
- U101 pad 7: (no net) -> /SCH101 Balanced Input and Differential Conversion/SCH101_L_LT5400_MINUS_SRC
- U101 pad 8: (no net) -> +18V
- U103 pad 1: /SCH101 Balanced Input and Differential Conversion/SCH101_L_LT5400_PLUS_SUM -> (no net)
- U103 pad 3: ROOT__PRE_EQ_L -> /SCH101 Balanced Input and Differential Conversion/SCH101_L_LT5400_PLUS_SUM
- U103 pad 4: +18V -> -18V
- U103 pad 5: -18V -> (no net)
- U103 pad 6: (no net) -> ROOT__PRE_EQ_L
- U103 pad 7: (no net) -> +18V
- U201 pad 1: Net-(U201-IN+) -> /SCH101 Balanced Input and Differential Conversion/SCH101_R_LT5400_PLUS_SRC
- U201 pad 2: Net-(U201-FB-) -> /SCH101 Balanced Input and Differential Conversion/SCH101_R_PLUS_FB
- U201 pad 3: /SCH101 Balanced Input and Differential Conversion/SCH101_R_LT5400_PLUS_SRC -> /SCH101 Balanced Input and Differential Conversion/SCH101_R_LOAD_POS
- U201 pad 4: +18V -> -18V
- U201 pad 5: -18V -> /SCH101 Balanced Input and Differential Conversion/SCH101_R_LOAD_NEG
- U201 pad 6: (no net) -> /SCH101 Balanced Input and Differential Conversion/SCH101_R_MINUS_FB
- U201 pad 7: (no net) -> /SCH101 Balanced Input and Differential Conversion/SCH101_R_LT5400_MINUS_SRC
- U201 pad 8: (no net) -> +18V
- U203 pad 1: /SCH101 Balanced Input and Differential Conversion/SCH101_R_LT5400_PLUS_SUM -> (no net)
- U203 pad 3: ROOT__PRE_EQ_R -> /SCH101 Balanced Input and Differential Conversion/SCH101_R_LT5400_PLUS_SUM
- U203 pad 4: +18V -> -18V
- U203 pad 5: -18V -> (no net)
- U203 pad 6: (no net) -> ROOT__PRE_EQ_R
- U203 pad 7: (no net) -> +18V
- U3001 pad 1: ROOT__PRE_EQ_L -> Net-(TP3002-TP)
- U3001 pad 3: Net-(TP3002-TP) -> ROOT__PRE_EQ_L
- U3001 pad 4: +18V -> -18V
- U3001 pad 5: -18V -> Net-(TP3003-TP)
- U3001 pad 6: (no net) -> Net-(U3001B-FB-)
- U3001 pad 7: (no net) -> Net-(TP3004-TP)
- U3001 pad 8: (no net) -> +18V
- U3501 pad 1: ROOT__PRE_EQ_R -> Net-(TP3502-TP)
- U3501 pad 3: Net-(TP3502-TP) -> ROOT__PRE_EQ_R
- U3501 pad 4: +18V -> -18V
- U3501 pad 5: -18V -> Net-(TP3503-TP)
- U3501 pad 6: (no net) -> Net-(U3501B-FB-)
- U3501 pad 7: (no net) -> Net-(TP3504-TP)
- U3501 pad 8: (no net) -> +18V
- U401 pad 1: ROOT__FILTERED_L -> Net-(U401A-IN-)
- U401 pad 2: Net-(U401-OUT) -> Net-(U401A-IN-)
- U401 pad 3: +18V -> ROOT__FILTERED_L
- U401 pad 5: 0VA -> ROOT__FILTERED_R
- U401 pad 6: (no net) -> Net-(U401B-IN-)
- U401 pad 7: (no net) -> Net-(U401B-IN-)
- U401 pad 8: (no net) -> +18V
- U501 pad 1: Net-(U501-IN) -> Net-(U501A-IN-)
- U501 pad 2: Net-(U501-OUT) -> Net-(U501A-IN-)
- U501 pad 3: +18V -> Net-(U501A-IN)
- U501 pad 5: 0VA -> Net-(U501B-IN)
- U501 pad 6: (no net) -> Net-(U501B-IN-)
- U501 pad 7: (no net) -> Net-(U501B-IN-)
- U501 pad 8: (no net) -> +18V
- U700 pad 1: Net-(U700-IN) -> Net-(TP7002-TP)
- U700 pad 3: +18V -> Net-(U700A-IN)
- U700 pad 5: 0VA -> Net-(U700B-IN)
- U700 pad 6: (no net) -> Net-(TP7003-TP)
- U700 pad 7: (no net) -> Net-(TP7003-TP)
- U700 pad 8: (no net) -> +18V
- U750 pad 1: Net-(U750-IN) -> Net-(TP7502-TP)
- U750 pad 3: +18V -> Net-(U750A-IN)
- U750 pad 5: 0VA -> Net-(U750B-IN)
- U750 pad 6: (no net) -> Net-(TP7503-TP)
- U750 pad 7: (no net) -> Net-(TP7503-TP)
- U750 pad 8: (no net) -> +18V
